File: HP3457A_NVSRAM_MOD.kicad_sch (KiCad schematic)
At the start: 15 parts, among them J1 Conn_01x02, U1 TC5564APL_Adapter, U2 STK12C68, U3 74AHC2G00, U4 TL431DBZ

Commit message: Moved to 0402 resistors, tweaked pours, minor cleanups.
Parts:
- R1, R5, R6: footprint Resistor_SMD:R_0603_1608Metric -> Resistor_SMD:R_0402_1005Metric_Pad0.72x0.64mm_HandSolder
- R2: value 530 -> 150; footprint Resistor_SMD:R_0603_1608Metric -> Resistor_SMD:R_0402_1005Metric_Pad0.72x0.64mm_HandSolder
- R3: value 1.5K -> 1.3K; footprint Resistor_SMD:R_0603_1608Metric -> Resistor_SMD:R_0402_1005Metric_Pad0.72x0.64mm_HandSolder
- R4: value 3.74K -> 3.3K; footprint Resistor_SMD:R_0603_1608Metric -> Resistor_SMD:R_0402_1005Metric_Pad0.72x0.64mm_HandSolder
Other:
- note added: "Two footprints to tune value See LTSpice simulation for R values"
- note removed: "Two footprints to tune value to 3.74K"
Changed lines of the file:
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@@
     (stroke (width 0) (type default) (color 0 0 0 0))
   )
-  (text "Two footprints to tune value to 3.74K" (at 68.58 177.8 0)
+  (text "Two footprints to tune value\nSee LTSpice simulation for R values"
+    (at 68.58 180.34 0)
     (effects (font (size 1.27 1.27)) (justify left bottom))
   )
@@
       (effects (font (size 1.27 1.27)) (justify left))
     )
-    (property "Value" "1.5K" (id 1) (at 70.3072 161.163 0)
-      (effects (font (size 1.27 1.27)) (justify left))
-    )
-    (property "Footprint" "Resistor_SMD:R_0603_1608Metric" (id 2) (at 69.596 160.274 90)
+    (property "Value" "1.3K" (id 1) (at 70.3072 161.163 0)
+      (effects (font (size 1.27 1.27)) (justify left))
+    )
+    (property "Footprint" "Resistor_SMD:R_0402_1005Metric_Pad0.72x0.64mm_HandSolder" (id 2) (at 69.596 160.274 90)
       (effects (font (size 1.27 1.27)) hide)
     )
@@
       (effects (font (size 1.27 1.27)) (justify left))
     )
-    (property "Value" "3.74K" (id 1) (at 70.3072 171.323 0)
-      (effects (font (size 1.27 1.27)) (justify left))
-    )
-    (property "Footprint" "Resistor_SMD:R_0603_1608Metric" (id 2) (at 69.596 170.434 90)
+    (property "Value" "3.3K" (id 1) (at 70.3072 171.323 0)
+      (effects (font (size 1.27 1.27)) (justify left))
+    )
+    (property "Footprint" "Resistor_SMD:R_0402_1005Metric_Pad0.72x0.64mm_HandSolder" (id 2) (at 69.596 170.434 90)
       (effects (font (size 1.27 1.27)) hide)
     )
@@
       (effects (font (size 1.27 1.27)) (justify left))
     )
-    (property "Value" "530" (id 1) (at 63.9572 151.003 0)
-      (effects (font (size 1.27 1.27)) (justify left))
-    )
-    (property "Footprint" "Resistor_SMD:R_0603_1608Metric" (id 2) (at 63.246 150.114 90)
+    (property "Value" "150" (id 1) (at 63.9572 151.003 0)
+      (effects (font (size 1.27 1.27)) (justify left))
+    )
+    (property "Footprint" "Resistor_SMD:R_0402_1005Metric_Pad0.72x0.64mm_HandSolder" (id 2) (at 63.246 150.114 90)
       (effects (font (size 1.27 1.27)) hide)
     )
@@
       (effects (font (size 1.27 1.27)) (justify left))
     )
-    (property "Footprint" "Resistor_SMD:R_0603_1608Metric" (id 2) (at 175.006 44.704 90)
+    (property "Footprint" "Resistor_SMD:R_0402_1005Metric_Pad0.72x0.64mm_HandSolder" (id 2) (at 175.006 44.704 90)
       (effects (font (size 1.27 1.27)) hide)
     )
@@
       (effects (font (size 1.27 1.27)) (justify left))
     )
-    (property "Footprint" "Resistor_SMD:R_0603_1608Metric" (id 2) (at 81.026 170.434 90)
+    (property "Footprint" "Resistor_SMD:R_0402_1005Metric_Pad0.72x0.64mm_HandSolder" (id 2) (at 81.026 170.434 90)
       (effects (font (size 1.27 1.27)) hide)
     )
@@
       (effects (font (size 1.27 1.27)) (justify left))
     )
-    (property "Footprint" "Resistor_SMD:R_0603_1608Metric" (id 2) (at 182.626 44.704 90)
+    (property "Footprint" "Resistor_SMD:R_0402_1005Metric_Pad0.72x0.64mm_HandSolder" (id 2) (at 182.626 44.704 90)
       (effects (font (size 1.27 1.27)) hide)
     )
@@
     )
     (path "/00000000-0000-0000-0000-0000635209b9"
-      (reference "R1") (unit 1) (value "10K") (footprint "Resistor_SMD:R_0603_1608Metric")
+      (reference "R1") (unit 1) (value "10K") (footprint "Resistor_SMD:R_0402_1005Metric_Pad0.72x0.64mm_HandSolder")
     )
     (path "/00000000-0000-0000-0000-00006344b67f"
-      (reference "R2") (unit 1) (value "530") (footprint "Resistor_SMD:R_0603_1608Metric")
+      (reference "R2") (unit 1) (value "150") (footprint "Resistor_SMD:R_0402_1005Metric_Pad0.72x0.64mm_HandSolder")
     )
     (path "/00000000-0000-0000-0000-00006344aae5"
-      (reference "R3") (unit 1) (value "1.5K") (footprint "Resistor_SMD:R_0603_1608Metric")
+      (reference "R3") (unit 1) (value "1.3K") (footprint "Resistor_SMD:R_0402_1005Metric_Pad0.72x0.64mm_HandSolder")
     )
     (path "/00000000-0000-0000-0000-00006344b517"
-      (reference "R4") (unit 1) (value "3.74K") (footprint "Resistor_SMD:R_0603_1608Metric")
+      (reference "R4") (unit 1) (value "3.3K") (footprint "Resistor_SMD:R_0402_1005Metric_Pad0.72x0.64mm_HandSolder")
     )
     (path "/ab748c29-941a-4289-898e-786b9fc4b780"
-      (reference "R5") (unit 1) (value "10K") (footprint "Resistor_SMD:R_0603_1608Metric")
+      (reference "R5") (unit 1) (value "10K") (footprint "Resistor_SMD:R_0402_1005Metric_Pad0.72x0.64mm_HandSolder")
     )
     (path "/071c3761-d773-432a-bdda-a9002a107f9e"
-      (reference "R6") (unit 1) (value "-") (footprint "Resistor_SMD:R_0603_1608Metric")
+      (reference "R6") (unit 1) (value "-") (footprint "Resistor_SMD:R_0402_1005Metric_Pad0.72x0.64mm_HandSolder")
     )
     (path "/00000000-0000-0000-0000-00006342de32"

Commit message: Design tweaked and gerbers submitted to OSHPark V1
Parts:
- renumbered U4 to U1, U1 to U10, U3 to U2, U2 to U3
Changed lines of the file:
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@@
   (symbol (lib_id "Memory_RAM_Toshiba:TC5564APL_Adapter") (at 66.04 67.31 0) (unit 1)
     (in_bom yes) (on_board yes)
-    (property "Reference" "U1" (id 0) (at 67.31 44.45 0)
+    (property "Reference" "U10" (id 0) (at 67.31 44.45 0)
       (effects (font (size 1.27 1.27)) (justify left))
     )
@@
   (symbol (lib_id "Memory_NVRAM_Cypress:STK12C68") (at 154.94 67.31 0) (unit 1)
     (in_bom yes) (on_board yes)
-    (property "Reference" "U2" (id 0) (at 156.21 44.45 0)
+    (property "Reference" "U3" (id 0) (at 156.21 44.45 0)
       (effects (font (size 1.27 1.27)) (justify left))
     )
@@
   (symbol (lib_id "Reference_Voltage:TL431DBZ") (at 62.23 165.1 270) (mirror x) (unit 1)
     (in_bom yes) (on_board yes)
-    (property "Reference" "U4" (id 0) (at 60.4774 163.9316 90)
+    (property "Reference" "U1" (id 0) (at 60.4774 163.9316 90)
       (effects (font (size 1.27 1.27)) (justify right))
     )
@@
   (symbol (lib_id "74xGxx:74AHC2G00") (at 97.79 73.66 0) (unit 1)
     (in_bom yes) (on_board yes)
-    (property "Reference" "U3" (id 0) (at 97.155 66.8782 0))
+    (property "Reference" "U2" (id 0) (at 97.155 66.8782 0))
     (property "Value" "74AHC2G00" (id 1) (at 97.155 69.1896 0))
     (property "Footprint" "Package_SO:TSSOP-8_3x3mm_P0.65mm" (id 2) (at 97.79 73.66 0)
@@
   (symbol (lib_id "74xGxx:74AHC2G00") (at 111.76 76.2 0) (unit 2)
     (in_bom yes) (on_board yes)
-    (property "Reference" "U3" (id 0) (at 109.22 80.01 0))
+    (property "Reference" "U2" (id 0) (at 109.22 80.01 0))
     (property "Value" "74AHC2G00" (id 1) (at 105.41 82.55 0))
     (property "Footprint" "Package_SO:TSSOP-8_3x3mm_P0.65mm" (id 2) (at 111.76 76.2 0)
@@
       (reference "R6") (unit 1) (value "-") (footprint "Resistor_SMD:R_0402_1005Metric_Pad0.72x0.64mm_HandSolder")
     )
+    (path "/00000000-0000-0000-0000-000063433874"
+      (reference "U1") (unit 1) (value "TL431DBZ") (footprint "Package_TO_SOT_SMD:SOT-23")
+    )
+    (path "/00000000-0000-0000-0000-00006348eea5"
+      (reference "U2") (unit 1) (value "74AHC2G00") (footprint "Package_SO:TSSOP-8_3x3mm_P0.65mm")
+    )
+    (path "/00000000-0000-0000-0000-00006349091b"
+      (reference "U2") (unit 2) (value "74AHC2G00") (footprint "Package_SO:TSSOP-8_3x3mm_P0.65mm")
+    )
+    (path "/00000000-0000-0000-0000-000063430085"
+      (reference "U3") (unit 1) (value "STK12C68") (footprint "Package_SO_Cypress:SOIC-28W_8.7x18.4mm_P1.27mm")
+    )
     (path "/00000000-0000-0000-0000-00006342de32"
-      (reference "U1") (unit 1) (value "TC5564APL_Adapter") (footprint "Package_DIP_Adapter:DIP-28_W15.24mm_Socket_Adapter")
-    )
-    (path "/00000000-0000-0000-0000-000063430085"
-      (reference "U2") (unit 1) (value "STK12C68") (footprint "Package_SO_Cypress:SOIC-28W_8.7x18.4mm_P1.27mm")
-    )
-    (path "/00000000-0000-0000-0000-00006348eea5"
-      (reference "U3") (unit 1) (value "74AHC2G00") (footprint "Package_SO:TSSOP-8_3x3mm_P0.65mm")
-    )
-    (path "/00000000-0000-0000-0000-00006349091b"
-      (reference "U3") (unit 2) (value "74AHC2G00") (footprint "Package_SO:TSSOP-8_3x3mm_P0.65mm")
-    )
-    (path "/00000000-0000-0000-0000-000063433874"
-      (reference "U4") (unit 1) (value "TL431DBZ") (footprint "Package_TO_SOT_SMD:SOT-23")
-    )
-  )
+      (reference "U10") (unit 1) (value "TC5564APL_Adapter") (footprint "Package_DIP_Adapter:DIP-28_W15.24mm_Socket_Adapter")
+    )
+  )

Commit message: Version submitted to OSHPark as V1
Parts:
- removed C2: 200nF, Capacitor_Tantalum_SMD:CP_EIA-6032-28_Kemet-C, symbol Device:C_Polarized_Small_US
- added C2, C5, C6, C7: 22u, Capacitor_SMD:C_0603_1608Metric, symbol Device:C_Small
- C1, C3, C4: Digikey 311-1087-1-ND -> 1276-1111-2-ND
- J1: MPN (none) -> XX62 nvSRAM V1
Connections:
- net GND: now also C2.2, C5.2, C6.2, C7.2
- net VCAP: now also C2.1, C5.1, C6.1, C7.1
Other:
- note added: "App note AN43593 Storage Capacitor (VCAP) Options for Infineon nvSRAM"
