File: 28PIN_6264_64K_NVSRAM_MOD/6264_NVSRAM_MOD.kicad_pcb (KiCad board)
At the start: 2 copper layers, 17.8 x 35.6 mm, 18 parts, among them J1 Conn_01x02, U1 TL431DBZ, U10 TC5564APL_Adapter, U2 74AHC2G00, U3 STK12C68

Commit message: Cleaned up some tiny offsets and a silkscreen bobble in 6264 NVSRAM board. Regenerated Gerbers.
Other:
- board text added: "V1B1"
- board text removed: "V1"
